File: Centralina_REV2.0/Centralina.kicad_pcb (KiCad board)
At the start: 4 copper layers, 239 parts, among them J1 Screw_Terminal_01x02, J10 Screw_Terminal_01x02, J11 Screw_Terminal_01x02, J12 Screw_Terminal_01x02, J13 Screw_Terminal_01x02, J14 Screw_Terminal_01x02, J15 Screw_Terminal_01x02, J16 Screw_Terminal_01x02, J17 Screw_Terminal_01x02, J18 Screw_Terminal_01x02, J19 Conn_02x04_Counter_Clockwise, J2 Screw_Terminal_01x02, J20 Conn_01x04_Pin, J3 Screw_Terminal_01x02, J4 Screw_Terminal_01x02, J5 Screw_Terminal_01x02, J6 Screw_Terminal_01x02, J7 Screw_Terminal_01x02, J8 Screw_Terminal_01x02, J9 Screw_Terminal_01x02, K1 SRD-05VDC-SL-C, K10 SRD-05VDC-SL-C, K11 SRD-05VDC-SL-C, K12 SRD-05VDC-SL-C, K13 SRD-05VDC-SL-C, K14 SRD-05VDC-SL-C, K15 SRD-05VDC-SL-C, K16 SRD-05VDC-SL-C, K2 SRD-05VDC-SL-C, K3 SRD-05VDC-SL-C, K4 SRD-05VDC-SL-C, K5 SRD-05VDC-SL-C, K6 SRD-05VDC-SL-C, K7 SRD-05VDC-SL-C, K8 SRD-05VDC-SL-C, K9 SRD-05VDC-SL-C, Q1 MMBT2222L, Q20 MMBT2222L, Q21 MMBT2222L, Q22 MMBT2222L, Q23 MMBT2222L, Q24 MMBT2222L, Q25 MMBT2222L, Q26 MMBT2222L, Q27 MMBT2222L, Q28 MMBT2222L, Q29 MMBT2222L, Q30 MMBT2222L, Q31 MMBT2222L, Q32 MMBT2222L, Q33 MMBT2222L, Q34 MMBT2222L, Q35 MMBT2222L, Q36 MMBT2222L, Q37 MMBT2222L, U1 LM2576HVS-5, U11 74HC14, U12 74HC14, U13 74HC14, U14 TPS7A0533PDBZ, U2 74HC00, U3 L7805, U4 L78L05_SOT89, U5 ULN2803A, U6 ULN2803A, U7 PCF8575DBR, U8 LM393, U9 PCF8575DBR

Commit message: Add files via upload
Parts:
- added C22: 1mF, Capacitor_THT:CP_Radial_D10.0mm_P5.00mm, F.Cu at (109.9, 46.5)
- BZ1: footprint Buzzer_Beeper:Indicator_PUI_AI-1440-TWT-24V-2-R -> JLCPCB_PART:BUZ-TH_BD9.0-P4.00-D0.6-FD
- C15: value 100uF -> 1mF
- C16: value 100uF -> 1mF; footprint Capacitor_SMD:CP_Elec_6.3x7.7 -> Capacitor_THT:CP_Radial_D10.0mm_P5.00mm
- C3: footprint Capacitor_SMD:CP_Elec_6.3x7.7 -> Capacitor_THT:CP_Radial_D5.0mm_P2.00mm
- J19: footprint Connector_PinSocket_2.54mm:PinSocket_2x04_P2.54mm_Vertical -> JLCPCB_PART:HDR-TH_8P-P2.54-V-F-R2-C4-S2.54
- J20: footprint Connector_PinSocket_2.54mm:PinSocket_1x04_P2.54mm_Horizontal -> JLCPCB_PART:HDR-TH_4P-P2.54-H-F-W10.2
- L1: footprint Inductor_SMD:L_Sunlord_MWSA1204S-1R0 -> JLCPCB_PART:IND-TH_BD13.0-P6.00-D0.8
- R108: footprint Resistor_THT:R_Axial_DIN0207_L6.3mm_D2.5mm_P10.16mm_Horizontal -> JLCPCB_PART:RES-TH_BD1.9-L3.3-P7.30-D0.5
- moved C16 35.6 mm to (73.3, 46.2)
- moved BZ1 18.7 mm to (134.3, 137.1)
- moved C21 13.8 mm to (128.9, 123.1)
- moved C24 13.8 mm to (128.9, 127.0)
- moved C20 12.6 mm to (125.5, 121.9)
- moved U14 12.6 mm to (125.5, 125.0)
- moved D19 11.6 mm to (111.1, 61.6), turned to -90 degrees
- moved R127 8.81 mm to (126.0, 115.2)
- moved C3 8.20 mm to (109.9, 52.1), turned to 0 degrees
- moved D18 7.21 mm to (115.9, 48.4)
- moved C7 5.06 mm to (105.5, 53.0)
- moved TP15 3.96 mm to (116.2, 46.5)
- moved R108 3.92 mm to (93.6, 158.0)
- moved J19 3.82 mm to (66.3, 116.6), turned to 90 degrees
- moved J20 3.81 mm to (115.4, 185.9), turned to 90 degrees
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Connections:
- C16 pad 1: /+5V -> /+12V_IN
- C21 pad 1: Net-(J19-Pin_5) -> Net-(J19-Pin_8)
- C24 pad 1: Net-(J19-Pin_5) -> Net-(J19-Pin_8)
- J19 pad 1: /Arduino_Core/MISO -> GND
- J19 pad 2: unconnected-(J19-Pin_8-Pad2) -> Net-(J19-Pin_8)
- J19 pad 3: /Arduino_Core/SCK -> /Arduino_Core/CE
- J19 pad 4: /Arduino_Core/MOSI -> /Arduino_Core/CSN
- J19 pad 5: /Arduino_Core/CE -> /Arduino_Core/SCK
- J19 pad 6: /Arduino_Core/CSN -> /Arduino_Core/MOSI
- J19 pad 7: GND -> /Arduino_Core/MISO
- J19 pad 8: Net-(J19-Pin_5) -> unconnected-(J19-Pin_5-Pad8)
- TP24 pad 1: Net-(J19-Pin_5) -> Net-(J19-Pin_8)
- U14 pad 2: Net-(J19-Pin_5) -> Net-(J19-Pin_8)
Routing:
- removed copper zone on In1.Cu, net GND
Other:
- copper layers 4 -> 2
