File: Centralina_REV2.0/Centralina.kicad_sch (KiCad schematic)
At the start: 12 parts, among them J16 Screw_Terminal_01x02, J17 Screw_Terminal_01x02, J18 Screw_Terminal_01x02, J19 Conn_02x04_Counter_Clockwise, J20 Conn_01x04_Pin, K16 SRD-05VDC-SL-C, U14 TPS7A0533PDBZ

Commit message: Add files via upload
Parts:
- added C16: 1mF, Capacitor_THT:CP_Radial_D10.0mm_P5.00mm, symbol Device:C_Polarized
- BZ1: footprint Buzzer_Beeper:Indicator_PUI_AI-1440-TWT-24V-2-R -> JLCPCB_PART:BUZ-TH_BD9.0-P4.00-D0.6-FD; REF C96102 -> C96256
- J19: footprint Connector_PinSocket_2.54mm:PinSocket_2x04_P2.54mm_Vertical -> JLCPCB_PART:HDR-TH_8P-P2.54-V-F-R2-C4-S2.54
- J20: footprint Connector_PinSocket_2.54mm:PinSocket_1x04_P2.54mm_Horizontal -> JLCPCB_PART:HDR-TH_4P-P2.54-H-F-W10.2
Connections:
- net +12V_IN: now also C16.1
- net Arduino_Core/CE: now also J19.3 (Pin_2); no longer J19.5 (Pin_3)
- net Arduino_Core/CSN: now also J19.4 (Pin_7); no longer J19.6 (Pin_6)
- net Arduino_Core/MISO: now also J19.7 (Pin_4); no longer J19.1 (Pin_1)
- net Arduino_Core/MOSI: now also J19.6 (Pin_6); no longer J19.4 (Pin_7)
- net Arduino_Core/SCK: now also J19.5 (Pin_3); no longer J19.3 (Pin_2)
- net GND: now also J19.1 (Pin_1), C16.2; no longer J19.7 (Pin_4)
- net at J19.2 (Pin_8): now also C21.1, C24.1, TP24.1, U14.2 (VO)
- now unconnected: J19.8 (Pin_5)
