File: Centralina_REV2.0/Modulo_Alimentazione.kicad_sch (KiCad schematic)
At the start: 41 parts, among them Q1 MMBT2222L, U1 LM2576HVS-5, U2 74HC00, U3 L7805, U4 L78L05_SOT89

Commit message: Add files via upload
Parts:
- removed C16: 100uF, Capacitor_SMD:CP_Elec_6.3x7.7, symbol Device:C_Polarized
- added C22: 1mF, Capacitor_THT:CP_Radial_D10.0mm_P5.00mm, symbol Device:C_Polarized
- C15: value 100uF -> 1mF; REF C503217 -> C88751
- C3: footprint Capacitor_SMD:CP_Elec_6.3x7.7 -> Capacitor_THT:CP_Radial_D5.0mm_P2.00mm; REF C72478 -> C43348
- L1: footprint Inductor_SMD:L_Sunlord_MWSA1204S-1R0 -> JLCPCB_PART:IND-TH_BD13.0-P6.00-D0.8; REF C408533 -> C5119631
Connections:
- net +5V_OUT: now also C22.1
- net GND: now also C22.2
Changed lines of the file:
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@@
 			)
 		)
-		(property "Value" "100uF"
+		(property "Value" "1mF"
 			(at 121.92 34.6709 0)
 			(effects
@@
 			)
 		)
-		(property "REF" "C503217"
+		(property "REF" "C88751"
 			(at 118.11 34.29 0)
 			(effects
@@
 	(symbol
 		(lib_id "Device:C_Polarized")
-		(at 234.95 34.29 0)
+		(at 248.92 34.29 0)
 		(unit 1)
 		(exclude_from_sim no)
@@
 		(dnp no)
 		(fields_autoplaced yes)
-		(property "Reference" "C3"
-			(at 238.76 32.1309 0)
+		(property "Reference" "C22"
+			(at 252.73 32.1309 0)
 			(effects
 				(font
@@
 			)
 		)
-		(property "Value" "100uF"
-			(at 238.76 34.6709 0)
+		(property "Value" "1mF"
+			(at 252.73 34.6709 0)
 			(effects
 				(font
@@
 			)
 		)
-		(property "Footprint" "Capacitor_SMD:CP_Elec_6.3x7.7"
-			(at 235.9152 38.1 0)
+		(property "Footprint" "Capacitor_THT:CP_Radial_D10.0mm_P5.00mm"
+			(at 249.8852 38.1 0)
 			(effects
 				(font
@@
 		)
 		(property "Datasheet" "~"
-			(at 234.95 34.29 0)
+			(at 248.92 34.29 0)
 			(effects
 				(font
@@
 		)
 		(property "Description" "Polarized capacitor"
-			(at 234.95 34.29 0)
+			(at 248.92 34.29 0)
 			(effects
 				(font
@@
 			)
 		)
-		(property "REF" "C72478"
-			(at 234.95 34.29 0)
+		(property "REF" "C88751"
+			(at 248.92 34.29 0)
 			(effects
 				(font
@@
 			(project "Centralina"
 				(path "/6c081a41-7694-4348-aefe-aafa0be843dc/300bbe2e-7418-4c1e-9996-603045772921"
-					(reference "C3")
+					(reference "C22")
 					(unit 1)
 				)
@@
 	)
 	(symbol
-		(lib_id "Regulator_Linear:L78L05_SOT89")
-		(at 111.76 66.04 0)
+		(lib_id "Device:C_Polarized")
+		(at 234.95 34.29 0)
 		(unit 1)
 		(exclude_from_sim no)
@@
 		(dnp no)
 		(fields_autoplaced yes)
-		(property "Reference" "U4"
-			(at 111.76 59.69 0)
+		(property "Reference" "C3"
+			(at 238.76 32.1309 0)
 			(effects
 				(font
 					(size 1.27 1.27)
 				)
+				(justify left)
 			)
 		)
-		(property "Value" "L78L05_SOT89"
-			(at 111.76 62.23 0)
+		(property "Value" "100uF"
+			(at 238.76 34.6709 0)
 			(effects
 				(font
 					(size 1.27 1.27)
 				)
+				(justify left)
 			)
 		)
-		(property "Footprint" "Package_TO_SOT_SMD:SOT-89-3"
-			(at 111.76 60.96 0)
+		(property "Footprint" "Capacitor_THT:CP_Radial_D5.0mm_P2.00mm"
+			(at 235.9152 38.1 0)
 			(effects
 				(font
 					(size 1.27 1.27)
-					(italic yes)
 				)
 				(hide yes)
 			)
 		)
-		(property "Datasheet" "http://www.st.com/content/ccc/resource/technical/document/datasheet/15/55/e5/aa/23/5b/43/fd/CD00000446.pdf/files/CD00000446.pdf/jcr:content/translations/en.CD00000446.pdf"
-			(at 111.76 67.31 0)
+		(property "Datasheet" "~"
+			(at 234.95 34.29 0)
 			(effects
 				(font
@@
 			)
 		)
-		(property "Description" "Positive 100mA 30V Linear Regulator, Fixed Output 5V, SOT-89"
-			(at 111.76 66.04 0)
+		(property "Description" "Polarized capacitor"
+			(at 234.95 34.29 0)
 			(effects
 				(font
@@
 			)
 		)
-		(property "REF" "C42738"
-			(at 111.76 66.04 0)
+		(property "REF" "C43348"
+			(at 234.95 34.29 0)
 			(effects
 				(font
@@
 			)
 		)
-		(pin "2"
-		)
 		(pin "1"
 		)
-		(pin "3"
+		(pin "2"
 		)
 		(instances
 			(project "Centralina"
 				(path "/6c081a41-7694-4348-aefe-aafa0be843dc/300bbe2e-7418-4c1e-9996-603045772921"
-					(reference "U4")
+					(reference "C3")
 					(unit 1)
 				)
@@
 	)
 	(symbol
-		(lib_id "Connector:TestPoint")
-		(at 64.77 52.07 270)
+		(lib_id "Regulator_Linear:L78L05_SOT89")
+		(at 111.76 66.04 0)
 		(unit 1)
 		(exclude_from_sim no)
@@
 		(dnp no)
 		(fields_autoplaced yes)
-		(property "Reference" "TP9"
-			(at 69.85 50.7999 90)
+		(property "Reference" "U4"
+			(at 111.76 59.69 0)
 			(effects
 				(font
 					(size 1.27 1.27)
 				)
-				(justify left)
 			)
 		)
-		(property "Value" "TestPoint"
-			(at 69.85 53.3399 90)
+		(property "Value" "L78L05_SOT89"
+			(at 111.76 62.23 0)
 			(effects
 				(font
 					(size 1.27 1.27)
 				)
-				(justify left)
 			)
 		)
-		(property "Footprint" "TestPoint:TestPoint_Pad_D1.0mm"
-			(at 64.77 57.15 0)
+		(property "Footprint" "Package_TO_SOT_SMD:SOT-89-3"
+			(at 111.76 60.96 0)
 			(effects
 				(font
 					(size 1.27 1.27)
+					(italic yes)
 				)
 				(hide yes)
 			)
 		)
-		(property "Datasheet" "~"
-			(at 64.77 57.15 0)
+		(property "Datasheet" "http://www.st.com/content/ccc/resource/technical/document/datasheet/15/55/e5/aa/23/5b/43/fd/CD00000446.pdf/files/CD00000446.pdf/jcr:content/translations/en.CD00000446.pdf"
+			(at 111.76 67.31 0)
 			(effects
 				(font
@@
 			)
 		)
-		(property "Description" "test point"
-			(at 64.77 52.07 0)
+		(property "Description" "Positive 100mA 30V Linear Regulator, Fixed Output 5V, SOT-89"
+			(at 111.76 66.04 0)
+			(effects
+				(font
+					(size 1.27 1.27)
+				)
+				(hide yes)
+			)
+		)
+		(property "REF" "C42738"
+			(at 111.76 66.04 0)
 			(effects
 				(font
@@
 			)
 		)
+		(pin "2"
+		)
 		(pin "1"
 		)
+		(pin "3"
+		)
 		(instances
 			(project "Centralina"
 				(path "/6c081a41-7694-4348-aefe-aafa0be843dc/300bbe2e-7418-4c1e-9996-603045772921"
-					(reference "TP9")
+					(reference "U4")
 					(unit 1)
 				)
@@
 	)
 	(symbol
-		(lib_id "Device:C_Polarized")
-		(at 248.92 34.29 0)
+		(lib_id "Connector:TestPoint")
+		(at 64.77 52.07 270)
 		(unit 1)
 		(exclude_from_sim no)
@@
 		(dnp no)
 		(fields_autoplaced yes)
-		(property "Reference" "C16"
-			(at 252.73 32.1309 0)
+		(property "Reference" "TP9"
+			(at 69.85 50.7999 90)
 			(effects
 				(font
@@
 			)
 		)
-		(property "Value" "100uF"
-			(at 252.73 34.6709 0)
+		(property "Value" "TestPoint"
+			(at 69.85 53.3399 90)
 			(effects
 				(font
@@
 			)
 		)
-		(property "Footprint" "Capacitor_SMD:CP_Elec_6.3x7.7"
-			(at 249.8852 38.1 0)
+		(property "Footprint" "TestPoint:TestPoint_Pad_D1.0mm"
+			(at 64.77 57.15 0)
 			(effects
 				(font
@@
 		)
 		(property "Datasheet" "~"
-			(at 248.92 34.29 0)
-			(effects
-				(font
-					(size 1.27 1.27)
-				)
-				(hide yes)
-			)
-		)
-		(property "Description" "Polarized capacitor"
-			(at 248.92 34.29 0)
+			(at 64.77 57.15 0)
 			(effects
 				(font
@@
 			)
 		)
-		(property "REF" "C72478"
-			(at 248.92 34.29 0)
+		(property "Description" "test point"
+			(at 64.77 52.07 0)
 			(effects
 				(font
@@
 		(pin "1"
 		)
-		(pin "2"
-		)
 		(instances
 			(project "Centralina"
 				(path "/6c081a41-7694-4348-aefe-aafa0be843dc/300bbe2e-7418-4c1e-9996-603045772921"
-					(reference "C16")
+					(reference "TP9")
 					(unit 1)
 				)
@@
 			)
 		)
-		(property "Footprint" "Inductor_SMD:L_Sunlord_MWSA1204S-1R0"
+		(property "Footprint" "JLCPCB_PART:IND-TH_BD13.0-P6.00-D0.8"
 			(at 106.68 27.94 0)
 			(effects
@@
 			)
 		)
-		(property "REF" "C408533"
+		(property "REF" "C5119631"
 			(at 106.68 27.94 0)
 			(effects
