File: Centralina_REV2.0/Trigger_IN.kicad_sch (KiCad schematic)
At the start: 28 parts, among them Q35 MMBT2222L, Q36 MMBT2222L, Q37 MMBT2222L, U8 LM393

Commit message: Add files via upload
Parts:
- R108: footprint Resistor_THT:R_Axial_DIN0207_L6.3mm_D2.5mm_P10.16mm_Horizontal -> JLCPCB_PART:RES-TH_BD1.9-L3.3-P7.30-D0.5
Changed lines of the file:
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@@
 			)
 		)
-		(property "Footprint" "Resistor_THT:R_Axial_DIN0207_L6.3mm_D2.5mm_P10.16mm_Horizontal"
+		(property "Footprint" "JLCPCB_PART:RES-TH_BD1.9-L3.3-P7.30-D0.5"
 			(at 97.79 46.228 90)
 			(effects
